File: kicad_V0/simplified_wiring_diagram.kicad_sch (KiCad schematic)
At the start: 17 parts, among them J5 USB_C_Receptacle_USB2.0_14P, J8 Conn_01x12_Pin, U12 SN74HC163N, U13 CD74HC4067M, U14 WEMOS_C3_mini, U15 CD74HC4067M, U16 SN74HC163N

Commit message: organised kicad files, with a separate V0
Parts:
- removed C2: 100n, symbol Device:C
- removed D10, D11, D12: WS2812B, LED_SMD:LED_WS2812B_PLCC4_5.0x5.0mm_P3.2mm, symbol LED:WS2812B
- removed D9: 1N4148, Diode_THT:D_DO-35_SOD27_P7.62mm_Horizontal, symbol Diode:1N4148
- removed J5: USB_C_Receptacle_USB2.0_14P, symbol Connector:USB_C_Receptacle_USB2.0_14P
- removed J8: Conn_01x12_Pin, symbol Connector:Conn_01x12_Pin
- removed R12, R13: 5.1K, symbol Device:R
- removed R14: 330, symbol Device:R
- removed R5: 3.3k, symbol Device:R
- removed RV3: 20k, symbol Device:R_Potentiometer_Trim
- removed U12, U16: SN74HC163N, SN74HC163N:DIP794W45P254L1969H508Q16, symbol SN74HC163N:SN74HC163N
- removed U13, U15: CD74HC4067M, Package_SO:SOIC-24W_7.5x15.4mm_P1.27mm, symbol 74xx:CD74HC4067M
- removed U14: WEMOS_C3_mini, RF_Module:WEMOS_C3_mini, symbol RF_Module:WEMOS_C3_mini
- added C1: 100n, symbol Device:C
- added D5: 1N4148, Diode_THT:D_DO-35_SOD27_P7.62mm_Horizontal, symbol Diode:1N4148
- added D6, D7, D8: WS2812B, LED_SMD:LED_WS2812B_PLCC4_5.0x5.0mm_P3.2mm, symbol LED:WS2812B
- added J4: USB_C_Receptacle_USB2.0_14P, symbol Connector:USB_C_Receptacle_USB2.0_14P
- added J6: Conn_01x10_Pin, symbol Connector:Conn_01x10_Pin
- added R10, R9: 5.1K, symbol Device:R
- added R11: 330, symbol Device:R
- added R4: 3.3k, symbol Device:R
- added RV2: 20k, symbol Device:R_Potentiometer_Trim
- added U10, U8: CD74HC4067M, Package_SO:SOIC-24W_7.5x15.4mm_P1.27mm, symbol 74xx:CD74HC4067M
- added U11, U4: SN74HC163N, SN74HC163N:DIP794W45P254L1969H508Q16, symbol SN74HC163N:SN74HC163N
- added U9: [GENERIC uC], RF_Module:WEMOS_C3_mini, symbol RF_Module:WEMOS_C3_mini
Connections:
- net +3.3V: now also J6.2 (Pin_2), U10.24 (VCC), U11.10 (ENT), U11.16 (VCC), U11.7 (ENP), U11.9 (~{LOAD}), U4.10 (ENT), U4.16 (VCC), U4.7 (ENP), U4.9 (~{LOAD}), U8.1 (COM), U8.24 (VCC), U9.8 (3V3)
- net +5V: now also D5.2 (A), D7.1 (VDD), D8.1 (VDD), J4.A4 (VBUS), J4.A9 (VBUS), J4.B4 (VBUS), J4.B9 (VBUS), J6.1 (Pin_1), U9.9 (VBus)
- net D0: now also C1.1, RV2.2, U10.1 (COM), U9.5 (D0)
- net D1: now also U4.2 (CLK), U9.4 (D1)
- net D10: now also R11.1, U9.14 (D10)
- net D2: now also U4.1 (~{CLR}), U9.3 (D2)
- net D3: now also U11.2 (CLK), U9.2 (D3)
- net D4: now also U11.1 (~{CLR}), U9.6 (D4)
- net D5: now also J6.4 (Pin_4), U9.7 (D5)
- net D6: now also J6.5 (Pin_5), U9.11 (D6)
- net D7: now also J6.6 (Pin_6), U9.12 (D7)
- net D8: now also J6.7 (Pin_7), U9.13 (D8)
- net EN: now also J6.10 (Pin_10), U9.1 (EN)
- net GND: now also C1.2, D6.3 (VSS), D7.3 (VSS), D8.3 (VSS), J4.A1 (GND), J4.A12 (GND), J4.B1 (GND), J4.B12 (GND), J4.SH (SHIELD), J6.3 (Pin_3), R10.1, R4.1, R9.2, U10.12 (GND), U10.15 (~{E}), U11.3 (A), U11.4 (B), U11.5 (C), U11.6 (D), U11.8 (GND), U4.3 (A), U4.4 (B), U4.5 (C), U4.6 (D), U4.8 (GND), U8.12 (GND), U8.15 (~{E}), U9.10 (GND)
- net RX: now also J6.8 (Pin_8), U9.15 (RX)
- net TX: now also J6.9 (Pin_9), U9.16 (TX)
- new net: D5.1 (K), D6.1 (VDD)
- new net: J4.B5 (CC2), R10.2
- new net: J4.A5 (CC1), R9.1
- new net: R4.2, RV2.3
- new net: U4.11 (QD), U8.13 (S3)
- new net: U4.12 (QC), U8.14 (S2)
- new net: U4.13 (QB), U8.11 (S1)
- new net: U4.14 (QA), U8.10 (S0)
- new net: D6.4 (DIN), R11.2
- new net: D7.2 (DOUT), D8.4 (DIN)
- new net: D6.2 (DOUT), D7.4 (DIN)
- new net: U10.13 (S3), U11.11 (QD)
- new net: U10.14 (S2), U11.12 (QC)
- new net: U10.11 (S1), U11.13 (QB)
- new net: U10.10 (S0), U11.14 (QA)
- no-connect marks 6 -> 7
Other:
- company: (none) -> By furballroller (Ayden Yak)
- title: (none) -> Super Cat Game
