File: kicad_V1/simplified_wiring_diagram.kicad_sch (KiCad schematic)
At the start: 14 parts, among them J3 USB_C_Receptacle_USB2.0_14P, U5 WEMOS_C3_mini, U6 CD74HC4067M, U7 CD74HC4067M

Commit message: organised kicad files, with a separate V0
Parts:
- U5: value WEMOS_C3_mini -> [GENERIC uC]
Other:
- note added: "Resistance of Velostat is read through a voltage divider"
Changed lines of the file:
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@@
 		(title "Super Cat Game")
 	)
-	(text_box "VELOSTAT (every possible handshake)"
-		(exclude_from_sim no)
-		(at 105.2717 176.53 90)
-		(size 3.9483 -40.64)
-		(margins 0.9525 0.9525 0.9525 0.9525)
+	(rectangle
+		(start 87.63 99.06)
+		(end 104.14 129.54)
 		(stroke
-			(width 0)
+			(width 0.4064)
 			(type solid)
+			(color 255 2 2 1)
 		)
 		(fill
 			(type none)
 		)
+	)
+	(rectangle
+		(start 88.9 78.74)
+		(end 95.25 88.9)
+		(stroke
+			(width 0.4064)
+			(type solid)
+			(color 255 2 2 1)
+		)
+		(fill
+			(type none)
+		)
+	)
+	(text "Resistance of Velostat\nis read through a\nvoltage divider"
+		(exclude_from_sim no)
+		(at 86.106 102.362 0)
 		(effects
 			(font
 				(size 1.27 1.27)
+				(thickness 0.254)
+				(bold yes)
+				(color 255 0 0 1)
 			)
-			(justify right top)
+			(justify right)
 		)
 	)
-	(text_box "Pin connections here are arbitrary (should suit pcb)"
+	(text_box "VELOSTAT (every possible handshake)"
 		(exclude_from_sim no)
-		(at 125.73 80.01 0)
-		(size 54.61 3.9483)
+		(at 105.2717 176.53 90)
+		(size 3.9483 -40.64)
 		(margins 0.9525 0.9525 0.9525 0.9525)
 		(stroke
@@
 				(size 1.27 1.27)
 			)
-			(justify left top)
+			(justify right top)
 		)
 	)
-	(text_box "NOT ENOUGH GPIO"
+	(text_box "Pin connections here are arbitrary (should suit pcb)"
 		(exclude_from_sim no)
-		(at 66.04 77.47 0)
-		(size 26.67 3.9483)
+		(at 125.73 80.01 0)
+		(size 54.61 3.9483)
 		(margins 0.9525 0.9525 0.9525 0.9525)
 		(stroke
@@
 		)
 		(instances
+			(project "circuit"
+				(path "/2ea3fbe2-2317-4d5c-acd1-47d626aa9ab4"
+					(reference "#PWR018")
+					(unit 1)
+				)
+			)
 			(project "pressure_sense"
 				(path "/edae9709-4638-4181-a40a-db9d181d67f1"
@@
 		)
 		(instances
+			(project "circuit"
+				(path "/2ea3fbe2-2317-4d5c-acd1-47d626aa9ab4"
+					(reference "R3")
+					(unit 1)
+				)
+			)
 			(project "pressure_sense"
 				(path "/edae9709-4638-4181-a40a-db9d181d67f1"
@@
 		)
 		(instances
+			(project "circuit"
+				(path "/2ea3fbe2-2317-4d5c-acd1-47d626aa9ab4"
+					(reference "R6")
+					(unit 1)
+				)
+			)
 			(project "pressure_sense"
 				(path "/edae9709-4638-4181-a40a-db9d181d67f1"
@@
 		)
 		(instances
+			(project "circuit"
+				(path "/2ea3fbe2-2317-4d5c-acd1-47d626aa9ab4"
+					(reference "C4")
+					(unit 1)
+				)
+			)
 			(project "pressure_sense"
 				(path "/edae9709-4638-4181-a40a-db9d181d67f1"
@@
 		)
 		(instances
+			(project "circuit"
+				(path "/2ea3fbe2-2317-4d5c-acd1-47d626aa9ab4"
+					(reference "R8")
+					(unit 1)
+				)
+			)
 			(project "pressure_sense"
 				(path "/edae9709-4638-4181-a40a-db9d181d67f1"
@@
 		)
 		(instances
+			(project "circuit"
+				(path "/2ea3fbe2-2317-4d5c-acd1-47d626aa9ab4"
+					(reference "J3")
+					(unit 1)
+				)
+			)
 			(project "pressure_sense"
 				(path "/edae9709-4638-4181-a40a-db9d181d67f1"
@@
 		)
 		(instances
+			(project "circuit"
+				(path "/2ea3fbe2-2317-4d5c-acd1-47d626aa9ab4"
+					(reference "U6")
+					(unit 1)
+				)
+			)
 			(project "pressure_sense"
 				(path "/edae9709-4638-4181-a40a-db9d181d67f1"
@@
 		)
 		(instances
+			(project "circuit"
+				(path "/2ea3fbe2-2317-4d5c-acd1-47d626aa9ab4"
+					(reference "D2")
+					(unit 1)
+				)
+			)
 			(project "pressure_sense"
 				(path "/edae9709-4638-4181-a40a-db9d181d67f1"
@@
 		)
 		(instances
+			(project "circuit"
+				(path "/2ea3fbe2-2317-4d5c-acd1-47d626aa9ab4"
+					(reference "#PWR017")
+					(unit 1)
+				)
+			)
 			(project "pressure_sense"
 				(path "/edae9709-4638-4181-a40a-db9d181d67f1"
@@
 			)
 		)
-		(property "Value" "WEMOS_C3_mini"
+		(property "Value" "[GENERIC uC]"
 			(at 81.28 67.818 90)
 			(show_name no)
@@
 		)
 		(instances
+			(project "circuit"
+				(path "/2ea3fbe2-2317-4d5c-acd1-47d626aa9ab4"
+					(reference "U5")
+					(unit 1)
+				)
+			)
 			(project "pressure_sense"
 				(path "/edae9709-4638-4181-a40a-db9d181d67f1"
@@
 		)
 		(instances
+			(project "circuit"
+				(path "/2ea3fbe2-2317-4d5c-acd1-47d626aa9ab4"
+					(reference "#PWR025")
+					(unit 1)
+				)
+			)
 			(project "pressure_sense"
 				(path "/edae9709-4638-4181-a40a-db9d181d67f1"
@@
 		)
 		(instances
+			(project "circuit"
+				(path "/2ea3fbe2-2317-4d5c-acd1-47d626aa9ab4"
+					(reference "#PWR026")
+					(unit 1)
+				)
+			)
 			(project "pressure_sense"
 				(path "/edae9709-4638-4181-a40a-db9d181d67f1"
@@
 		)
 		(instances
+			(project "circuit"
+				(path "/2ea3fbe2-2317-4d5c-acd1-47d626aa9ab4"
+					(reference "D4")
+					(unit 1)
+				)
+			)
 			(project "pressure_sense"
 				(path "/edae9709-4638-4181-a40a-db9d181d67f1"
@@
 		)
 		(instances
+			(project "circuit"
+				(path "/2ea3fbe2-2317-4d5c-acd1-47d626aa9ab4"
+					(reference "D1")
+					(unit 1)
+				)
+			)
 			(project "pressure_sense"
 				(path "/edae9709-4638-4181-a40a-db9d181d67f1"
@@
 		)
 		(instances
+			(project "circuit"
+				(path "/2ea3fbe2-2317-4d5c-acd1-47d626aa9ab4"
+					(reference "#PWR011")
+					(unit 1)
+				)
+			)
 			(project "pressure_sense"
 				(path "/edae9709-4638-4181-a40a-db9d181d67f1"
@@
 		)
 		(instances
+			(project "circuit"
+				(path "/2ea3fbe2-2317-4d5c-acd1-47d626aa9ab4"
+					(reference "#PWR015")
+					(unit 1)
+				)
+			)
 			(project "pressure_sense"
 				(path "/edae9709-4638-4181-a40a-db9d181d67f1"
@@
 		)
 		(instances
+			(project "circuit"
+				(path "/2ea3fbe2-2317-4d5c-acd1-47d626aa9ab4"
+					(reference "#PWR030")
+					(unit 1)
+				)
+			)
 			(project "pressure_sense"
 				(path "/edae9709-4638-4181-a40a-db9d181d67f1"
@@
 		)
 		(instances
+			(project "circuit"
+				(path "/2ea3fbe2-2317-4d5c-acd1-47d626aa9ab4"
+					(reference "#PWR027")
+					(unit 1)
+				)
+			)
 			(project "pressure_sense"
 				(path "/edae9709-4638-4181-a40a-db9d181d67f1"
@@
 		)
 		(instances
+			(project "circuit"
+				(path "/2ea3fbe2-2317-4d5c-acd1-47d626aa9ab4"
+					(reference "D3")
+					(unit 1)
+				)
+			)
 			(project "pressure_sense"
 				(path "/edae9709-4638-4181-a40a-db9d181d67f1"
@@
 		)
 		(instances
+			(project "circuit"
+				(path "/2ea3fbe2-2317-4d5c-acd1-47d626aa9ab4"
+					(reference "#PWR029")
+					(unit 1)
+				)
+			)
 			(project "pressure_sense"
 				(path "/edae9709-4638-4181-a40a-db9d181d67f1"
@@
 		)
 		(instances
+			(project "circuit"
+				(path "/2ea3fbe2-2317-4d5c-acd1-47d626aa9ab4"
+					(reference "R7")
+					(unit 1)
+				)
+			)
 			(project "pressure_sense"
 				(path "/edae9709-4638-4181-a40a-db9d181d67f1"
@@
 		)
 		(instances
+			(project "circuit"
+				(path "/2ea3fbe2-2317-4d5c-acd1-47d626aa9ab4"
+					(reference "#PWR016")
+					(unit 1)
+				)
+			)
 			(project "pressure_sense"
 				(path "/edae9709-4638-4181-a40a-db9d181d67f1"
@@
 		)
 		(instances
+			(project "circuit"
+				(path "/2ea3fbe2-2317-4d5c-acd1-47d626aa9ab4"
+					(reference "RV1")
+					(unit 1)
+				)
+			)
 			(project "pressure_sense"
 				(path "/edae9709-4638-4181-a40a-db9d181d67f1"
@@
 		)
 		(instances
+			(project "circuit"
+				(path "/2ea3fbe2-2317-4d5c-acd1-47d626aa9ab4"
+					(reference "U7")
+					(unit 1)
+				)
+			)
 			(project "pressure_sense"
 				(path "/edae9709-4638-4181-a40a-db9d181d67f1"
@@
 		)
 		(instances
+			(project "circuit"
+				(path "/2ea3fbe2-2317-4d5c-acd1-47d626aa9ab4"
+					(reference "#PWR012")
+					(unit 1)
+				)
+			)
 			(project "pressure_sense"
 				(path "/edae9709-4638-4181-a40a-db9d181d67f1"
@@
 		)
 		(instances
+			(project "circuit"
+				(path "/2ea3fbe2-2317-4d5c-acd1-47d626aa9ab4"
+					(reference "#PWR0107")
+					(unit 1)
+				)
+			)
 			(project "pressure_sense"
 				(path "/edae9709-4638-4181-a40a-db9d181d67f1"
@@
 		)
 		(instances
+			(project "circuit"
+				(path "/2ea3fbe2-2317-4d5c-acd1-47d626aa9ab4"
+					(reference "#PWR010")
+					(unit 1)
+				)
+			)
 			(project "pressure_sense"
 				(path "/edae9709-4638-4181-a40a-db9d181d67f1"
